Commit message: Add end effector link to robot model

File: src/summer_robotics/urdf/simple_robot.urdf (robot description, URDF)
Before this commit: robot two_link_robot, 3 links, 2 joints
Links:
- added link end_effector_link, mass 0.1; collision cylinder length=0.15 radius=0.03; visual cylinder length=0.15 radius=0.03
- added link world
Joints:
- added joint end_effector_fixed_joint: type fixed, parent link_2, child end_effector_link, origin xyz=0 0 0.8 rpy=0 0 0
- added joint world_to_base: type fixed, parent world, child base_link, origin xyz=0 0 0 rpy=0 0 0
- joint joint_2: limit lower=-1.57 upper=1.57 effort=10 velocity=1.0 -> lower=-2.5 upper=2.5 effort=10 velocity=1.0

Commit message: Fix Gazebo ros2 control and restore robot motion

File: src/summer_robotics/urdf/simple_robot.urdf (robot description, URDF)
Before this commit: robot two_link_robot, 5 links, 4 joints
Links:
- removed link world
- link base_link: mass 2.0 -> 20.0
Joints:
- removed joint world_to_base
- joint joint_1: limit lower=-1.57 upper=1.57 effort=10 velocity=1.0 -> lower=-1.57 upper=1.57 effort=100 velocity=1.0
- joint joint_2: limit lower=-2.5 upper=2.5 effort=10 velocity=1.0 -> lower=-2.5 upper=2.5 effort=100 velocity=1.0

Commit message: Add base yaw joint and 3D reaching support

File: src/summer_robotics/urdf/simple_robot.urdf (robot description, URDF)
Before this commit: robot two_link_robot, 4 links, 3 joints
Links:
- added link yaw_link, mass 1.0; collision cylinder length=0.10 radius=0.08; visual cylinder length=0.10 radius=0.08
Joints:
- added joint joint_0: type revolute, parent base_link, child yaw_link, origin xyz=0 0 0.1 rpy=0 0 0, axis 0 0 1, limit lower=-3.14 upper=3.14 effort=100 velocity=1.0
- joint joint_1: parent base_link -> yaw_link

Commit message: Add gripper control for pick and place

File: src/summer_robotics/urdf/simple_robot.urdf (robot description, URDF)
Before this commit: robot two_link_robot, 5 links, 4 joints
Links:
- added link gripper_link, mass 0.1; collision box size=0.12 0.03 0.08; visual box size=0.12 0.03 0.08
Joints:
- added joint gripper_joint: type prismatic, parent end_effector_link, child gripper_link, origin xyz=0 0 0.15 rpy=0 0 0, axis 0 1 0, limit lower=0.0 upper=0.04 effort=20 velocity=0.1
